Commit message: taihu support

File: description/robots/N2/urdf/N2.urdf (robot description, URDF)
Before this commit: robot N2, 19 links, 18 joints
Links:
- added link L_arm_hand_Link, mass 0.063335; collision mesh filename=../meshes/l_arm_hand_Link.STL; visual mesh filename=../meshes/l_arm_hand_Link.STL
- added link R_arm_hand_link, mass 0.063335; collision mesh filename=../meshes/r_arm_hand_Link.STL; visual mesh filename=../meshes/r_arm_hand_Link.STL
Joints:
- added joint L_arm_hand_joint: type , parent L_arm_elbow_Link, child L_arm_hand_Link, origin xyz=-0.0045 0.00036368 -0.1815 rpy=0 0 0, axis 0 0 0
- added joint R_arm_hand_joint: type , parent R_arm_elbow_Link, child R_arm_hand_link, origin xyz=-0.0045 0.00018648 -0.18067 rpy=0 0 0, axis 0 0 0

Commit message: N2

File: description/robots/N2/urdf/N2.urdf (robot description, URDF)
Before this commit: robot N2, 21 links, 20 joints
Joints:
- joint L_arm_hand_joint: type  -> fixed
- joint R_arm_hand_joint: type  -> fixed

Commit message: N2

File: description/robots/N2/urdf/N2.urdf (robot description, URDF)
Before this commit: robot N2, 21 links, 20 joints
Joints:
- joint R_arm_shoulder_pitch_joint: axis 0 0 -1 -> 0 0 1
